File: pcb/cc_proto.sch (KiCad schematic (older format))
At the start: 39 parts, among them SW1 SW_PUSH, SW10 SW_PUSH, SW11 SW_PUSH, SW12 SW_PUSH, SW13 SW_PUSH, SW14 SW_PUSH, SW15 SW_PUSH, SW16 SW_PUSH, SW17 SW_PUSH, SW18 SW_PUSH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

Commit message: PCB Rev.4
Parts:
- D1, D10, D11, D12, D13, D14, D15, D16, D17, D18, D2, D3, D4, D5, D6, D7, D8, D9: footprint cc_proto:D3_TH_SMD -> cc_proto:D3_TH_SMD_Text-Added
- LED1: footprint cc_proto:SK6812MINI_rev -> cc_proto:SK6812MINI_rev_Text-Added
- SW1, SW10, SW11, SW12, SW13, SW14, SW15, SW16, SW17, SW18, SW2, SW3, SW4, SW5, SW6, SW7, SW8, SW9: footprint cc_proto:CherryMX_MidHeight_Hotswap_Choc12_Alps -> cc_proto:CherryMX_MidHeight_Hotswap_Choc12_Alps_v2
- U1: footprint cc_proto:ProMicro_v2 -> cc_proto:ProMicro_v2_Text-Changed
